Commit message: feat(sim): Ensamble del brazo robótico sobre el chasis de Maya

File: AutoNav_Mission_2026/src/maya_description/urdf/maya_description.urdf.xacro (robot description, xacro)
@@ -9,3 +9,7 @@
   <xacro:include filename="$(find maya_description)/urdf/sensors.xacro"/>
   <xacro:include filename="$(find maya_description)/urdf/maya_arm_mount.xacro"/>
+  <xacro:include filename="$(find maya_description)/urdf/maya_arm.xacro"/>
+  <xacro:maya_arm parent="maya_arm_mount">
+    <origin xyz="0 0 0" rpy="0 0 0"/>
+  </xacro:maya_arm>
 </robot>
