Commit message: Subir copia funcional de la simulacion AutoNav_Mission_2026 a main

File: AutoNav_Mission_2026/src/maya_description/urdf/arm_base.xacro (robot description, xacro)
@@ -1,32 +1,25 @@
 <?xml version="1.0" encoding="utf-8"?>
 <robot xmlns:xacro="http://www.ros.org/wiki/xacro">
-  <xacro:macro name="maya_arm" params="parent *origin">
-    <!-- Joint dinámico para atornillar el brazo al Rover -->
-    <joint name="arm_mount_joint" type="fixed">
-      <xacro:insert_block name="origin" />
-      <parent link="${parent}" />
-      <child link="arm_base_link" />
-    </joint>
-    <link name="arm_base_link">
-      <inertial>
-        <origin xyz="1.281E-06 -0.015414 0.0001483" rpy="0 0 0" />
-        <mass value="0.13795" />
-        <inertia ixx="5.7399E-05" ixy="-2.5472E-09" ixz="1.5566E-09" iyy="9.0274E-05" iyz="3.1683E-07" izz="5.7877E-05" />
-      </inertial>
-      <visual>
-        <origin xyz="0 0 0" rpy="0 0 0" />
-        <geometry>
-          <mesh filename="package://maya_description/meshes/base_link_arm.STL" />
-        </geometry>
-        <material name=""><color rgba="0.25098 0.25098 0.25098 1" /></material>
-      </visual>
-      <collision>
-        <origin xyz="0 0 0" rpy="0 0 0" />
-        <geometry>
-          <mesh filename="package://maya_description/meshes/base_link_arm.STL" />
-        </geometry>
-      </collision>
-    </link>
-    <link name="motor_1_link">
+  <link name="arm_base_link">
+    <inertial>
+      <origin xyz="1.281E-06 -0.015414 0.0001483" rpy="0 0 0" />
+      <mass value="0.13795" />
+      <inertia ixx="5.7399E-05" ixy="-2.5472E-09" ixz="1.5566E-09" iyy="9.0274E-05" iyz="3.1683E-07" izz="5.7877E-05" />
+    </inertial>
+    <visual>
+      <origin xyz="0 0 0" rpy="0 0 0" />
+      <geometry>
+        <mesh filename="package://maya_description/meshes/base_link_arm.STL" />
+      </geometry>
+      <material name=""><color rgba="0.25098 0.25098 0.25098 1" /></material>
+    </visual>
+    <collision>
+      <origin xyz="0 0 0" rpy="0 0 0" />
+      <geometry>
+        <mesh filename="package://maya_description/meshes/base_link_arm.STL" />
+      </geometry>
+    </collision>
+  </link>
+  <link name="motor_1_link">
     <inertial>
       <origin
@@ -317,4 +310,3 @@
       velocity="0" />
   </joint>
-  </xacro:macro>
 </robot>

File: AutoNav_Mission_2026/src/maya_description/urdf/common_properties.xacro (robot description, xacro)
@@ -53,5 +53,5 @@
   <xacro:property name="wheel_inertia_iyz" value="-9.6151E-08"/>
   <xacro:property name="wheel_inertia_izz" value="0.025537"/>
-  <!--Origen de la conexion Maya|Brazo-->
+  <!--Origen de la base Maya|Brazo-->
   <xacro:property name="maya_arm_mount_xyz" value="0 -0.386 0.052"/>
   <xacro:property name="maya_arm_mount_rpy" value="0 0 0"/>
@@ -121,5 +121,5 @@
   <xacro:property name="drive_wheel_separation" value="1.09449"/>
   <xacro:property name="drive_wheel_radius"     value="0.1636"/>
-<!-- Macro para las paredes del brazo -->
+<!-- Macro para las paredes del maya | brazo -->
   <xacro:macro name="arm_wall" params="link_name joint_name xyz rpy">
     <link name="${link_name}">

File: AutoNav_Mission_2026/src/maya_description/urdf/maya_arm_mount.xacro (robot description, xacro)
@@ -2,17 +2,17 @@
 <robot xmlns:xacro="http://www.ros.org/wiki/xacro">
 <!--Paredes de Brazo-->
-<!--Pared Derecha-->
-<xacro:arm_wall
-    link_name="arm_wall_right"
-    joint_name="arm_wall_right_joint"
-    xyz="${arm_wall_right_xyz}"
-    rpy="${arm_wall_right_rpy}"/>
-<!--Pared Izquieda-->
-<xacro:arm_wall
-    link_name="arm_wall_left"
-    joint_name="arm_wall_left_joint"
-    xyz="${arm_wall_left_xyz}"
-    rpy="${arm_wall_left_rpy}"/>
-<!--Fixed conexion Maya|Brazo-->
+    <!--Pared Derecha-->
+    <xacro:arm_wall
+        link_name="arm_wall_right"
+        joint_name="arm_wall_right_joint"
+        xyz="${arm_wall_right_xyz}"
+        rpy="${arm_wall_right_rpy}"/>
+    <!--Pared Izquieda-->
+    <xacro:arm_wall
+        link_name="arm_wall_left"
+        joint_name="arm_wall_left_joint"
+        xyz="${arm_wall_left_xyz}"
+        rpy="${arm_wall_left_rpy}"/>
+    <!--Fixed conexion Maya|Brazo-->
     <link name="maya_arm_mount">
         <visual>
@@ -24,4 +24,5 @@
         </visual>
     </link>
+<!-- Base para brazo y laboratorio en Maya -->
     <joint name="maya_arm_mount_joint" type="fixed">
         <parent link="base_link"/>
@@ -29,3 +30,9 @@
         <origin xyz="${maya_arm_mount_xyz}" rpy="${maya_arm_mount_rpy}"/>
     </joint>
+<!-- Joint para atornillar el brazo a Maya -->
+    <joint name="arm_mount_joint" type="fixed">
+      <parent link="maya_arm_mount" />
+      <child link="arm_base_link" />
+      <origin xyz="${arm_mount_xyz}" rpy="${arm_mount_rpy}"/>
+    </joint>
 </robot>

File: AutoNav_Mission_2026/src/maya_description/urdf/maya_description.urdf.xacro (robot description, xacro)
@@ -1,5 +1,4 @@
 <?xml version="1.0"?>
-<robot name="maya"
-  xmlns:xacro="http://www.ros.org/wiki/xacro">
+<robot xmlns:xacro="http://www.ros.org/wiki/xacro">
   <!-- brief Top level robot description for Maya Rover -->
   <!-- This file aggregates shared properties, physical model and Gazebo plugins -->
@@ -8,8 +7,3 @@
   <xacro:include filename="$(find maya_description)/urdf/mobile_base_gazebo.xacro"/>
   <xacro:include filename="$(find maya_description)/urdf/sensors.xacro"/>
-  <xacro:include filename="$(find maya_description)/urdf/maya_arm_mount.xacro"/>
-  <xacro:include filename="$(find maya_description)/urdf/maya_arm.xacro"/>
-  <xacro:maya_arm parent="maya_arm_mount">
-    <origin xyz="0 0 0" rpy="0 0 0"/>
-  </xacro:maya_arm>
 </robot>

Commit message: stl optimizados y frame zed

File: AutoNav_Mission_2026/src/maya_description/urdf/arm_base.xacro (robot description, xacro)
@@ -64,5 +64,5 @@
     type="revolute">
     <origin
-      xyz="0 0.01 0"
+      xyz="0.01 0.01 0"
       rpy="1.6654 0.083193 2.1147" />
     <parent
@@ -73,8 +73,8 @@
       xyz="0.083097 -0.99208 0.094171" />
     <limit
-      lower="0"
-      upper="0"
-      effort="0"
-      velocity="0" />
+      lower="-3.14"
+      upper="3.14"
+      effort="10"
+      velocity="1" />
   </joint>
   <link
@@ -131,8 +131,8 @@
       xyz="0.95882 0.10535 0.26374" />
     <limit
-      lower="0"
-      upper="0"
-      effort="0"
-      velocity="0" />
+      lower="-1.57"
+      upper="1.57"
+      effort="10"
+      velocity="1" />
   </joint>
   <link
@@ -189,8 +189,8 @@
       xyz="0.95882 0.10535 0.26374" />
     <limit
-      lower="0"
-      upper="0"
-      effort="0"
-      velocity="0" />
+      lower="-2.09"
+      upper="2.09"
+      effort="10"
+      velocity="1" />
   </joint>
   <link
@@ -247,8 +247,8 @@
       xyz="0.95882 0.10535 0.26374" />
     <limit
-      lower="0"
-      upper="0"
-      effort="0"
-      velocity="0" />
+      lower="-2.62"
+      upper="2.62"
+      effort="10"
+      velocity="1" />
   </joint>
   <link
@@ -305,8 +305,8 @@
       xyz="0.099071 0.74625 -0.65825" />
     <limit
-      lower="0"
-      upper="0"
-      effort="0"
-      velocity="0" />
+      lower="-3.14"
+      upper="3.14"
+      effort="10"
+      velocity="1" />
   </joint>
 </robot>

File: AutoNav_Mission_2026/src/maya_description/urdf/arm_properties.xacro (robot description, xacro)
@@ -2,5 +2,5 @@
 <robot xmlns:xacro="http://www.ros.org/wiki/xacro">
   <!--Origen del Frame para atornillar el brazo en Maya-->
-  <xacro:property name="arm_mount_xyz" value="0 0 0.04"/>
+  <xacro:property name="arm_mount_xyz" value="-0 0 0.04"/>
   <xacro:property name="arm_mount_rpy" value="0 0 0"/>
 </robot>

File: AutoNav_Mission_2026/src/maya_description/urdf/common_properties.xacro (robot description, xacro)
@@ -7,4 +7,7 @@
   <material name="maya_wheel">
     <color rgba="0.05 0.05 0.05 1.0"/>
+  </material>
+  <material name="sensors">
+    <color rgba="0.2 0 0.2 1"/>
   </material>
   <!-- Mesh scale factor for all STL geometry.
@@ -53,5 +56,5 @@
   <xacro:property name="wheel_inertia_iyz" value="-9.6151E-08"/>
   <xacro:property name="wheel_inertia_izz" value="0.025537"/>
-  <!--Origen de la base Maya|Brazo-->
+  <!--Origen de la base Maya | Brazo-->
   <xacro:property name="maya_arm_mount_xyz" value="0 -0.386 0.052"/>
   <xacro:property name="maya_arm_mount_rpy" value="0 0 0"/>

File: AutoNav_Mission_2026/src/maya_description/urdf/mobile_base.xacro (robot description, xacro)
@@ -18,5 +18,6 @@
       <origin xyz="${base_link_mesh_offset_xyz}" rpy="${base_link_mesh_offset_rpy}"/>
       <geometry>
-        <mesh filename="file://$(find maya_description)/meshes/base_link.STL" scale="${mesh_scale} ${mesh_scale} ${mesh_scale}"/>
+        <!--mesh filename="file://$(find maya_description)/meshes/base_link.STL" scale="${mesh_scale} ${mesh_scale} ${mesh_scale}"/-->
+        <mesh filename="file://$(find maya_description)/meshes/optimized/base_link_optimized/base_link_keep025.stl" scale="${mesh_scale} ${mesh_scale} ${mesh_scale}"/>
       </geometry>
       <material name="maya_body"/>
@@ -25,5 +26,6 @@
       <origin xyz="${base_link_mesh_offset_xyz}" rpy="${base_link_mesh_offset_rpy}"/>
       <geometry>
-        <mesh filename="file://$(find maya_description)/meshes/base_link.STL" scale="${mesh_scale} ${mesh_scale} ${mesh_scale}"/>
+        <!--mesh filename="file://$(find maya_description)/meshes/base_link.STL" scale="${mesh_scale} ${mesh_scale} ${mesh_scale}"/-->
+        <mesh filename="file://$(find maya_description)/meshes/optimized/base_link_optimized/base_link_keep002.stl" scale="${mesh_scale} ${mesh_scale} ${mesh_scale}"/>
       </geometry>
     </collision>
@@ -80,8 +82,18 @@
        float or overload another during skid-steer turns. -->
   <!-- Left wheels use default spin axis from wheel_axis_left -->
-  <xacro:maya_wheel prefix="front_left" mesh="file://$(find maya_description)/meshes/front_left.STL" xyz="-0.32478 -0.62736 -0.2764" rpy="1.5702 0 1.5708" inertial_xyz="-4.8481E-06 -8.0801E-06 -0.057753" inertial_rpy="0 0 0"/>
-  <xacro:maya_wheel prefix="back_left" mesh="file://$(find maya_description)/meshes/back_left.STL" xyz="-0.32513 0.28848 -0.2764" rpy="1.5708 0 1.5708" inertial_xyz="-4.8481E-06 -8.0801E-06 -0.057572" inertial_rpy="0 0 0"/>
+<!--
+Original
+  |
+  v
+Copia
+-->
+  <!--xacro:maya_wheel prefix="front_left" mesh="file://$(find maya_description)/meshes/front_left.STL" xyz="-0.32478 -0.62736 -0.2764" rpy="1.5702 0 1.5708" inertial_xyz="-4.8481E-06 -8.0801E-06 -0.057753" inertial_rpy="0 0 0"/-->
+  <xacro:maya_wheel prefix="front_left" mesh="file://$(find maya_description)/meshes/optimized/front_left_optimized/front_left_keep025.stl" xyz="-0.32478 -0.62736 -0.2764" rpy="1.5702 0 1.5708" inertial_xyz="-4.8481E-06 -8.0801E-06 -0.057753" inertial_rpy="0 0 0"/>
+  <!--xacro:maya_wheel prefix="back_left" mesh="file://$(find maya_description)/meshes/back_left.STL" xyz="-0.32513 0.28848 -0.2764" rpy="1.5708 0 1.5708" inertial_xyz="-4.8481E-06 -8.0801E-06 -0.057572" inertial_rpy="0 0 0"/-->
+  <xacro:maya_wheel prefix="back_left" mesh="file://$(find maya_description)/meshes/optimized/back_left_optimized/back_left_keep025.stl" xyz="-0.32513 0.28848 -0.2764" rpy="1.5708 0 1.5708" inertial_xyz="-4.8481E-06 -8.0801E-06 -0.057572" inertial_rpy="0 0 0"/>
   <!-- Right wheels override spin axis to wheel_axis_right -->
-  <xacro:maya_wheel prefix="front_right" mesh="file://$(find maya_description)/meshes/front_right.STL" xyz="0.3112596 -0.61714 -0.2764" rpy="1.5657 0.51887 -1.5734" axis="${wheel_axis_right}" inertial_xyz="-4.8512E-06 -8.0627E-06 -0.046342" inertial_rpy="0 0 0"/>
-  <xacro:maya_wheel prefix="back_right" mesh="file://$(find maya_description)/meshes/back_right.STL" xyz="0.3112382 0.27364 -0.2764" rpy="-1.5781 -0.91737 1.5766" axis="${wheel_axis_right}" inertial_xyz="-4.8659E-06 -8.069E-06 -0.034709" inertial_rpy="0 0 0"/>
+  <!--xacro:maya_wheel prefix="front_right" mesh="file://$(find maya_description)/meshes/front_right.STL" xyz="0.3112596 -0.61714 -0.2764" rpy="1.5657 0.51887 -1.5734" axis="${wheel_axis_right}" inertial_xyz="-4.8512E-06 -8.0627E-06 -0.046342" inertial_rpy="0 0 0"/-->
+  <xacro:maya_wheel prefix="front_right" mesh="file://$(find maya_description)/meshes/optimized/front_right_optimized/front_right_keep025.stl" xyz="0.3112596 -0.61714 -0.2764" rpy="1.5657 0.51887 -1.5734" axis="${wheel_axis_right}" inertial_xyz="-4.8512E-06 -8.0627E-06 -0.046342" inertial_rpy="0 0 0"/>
+  <!--xacro:maya_wheel prefix="back_right" mesh="file://$(find maya_description)/meshes/back_right.STL" xyz="0.3112382 0.27364 -0.2764" rpy="-1.5781 -0.91737 1.5766" axis="${wheel_axis_right}" inertial_xyz="-4.8659E-06 -8.069E-06 -0.034709" inertial_rpy="0 0 0"/-->
+  <xacro:maya_wheel prefix="back_right" mesh="file://$(find maya_description)/meshes/optimized/back_right_optimized/back_right_keep025.stl" xyz="0.3112382 0.27364 -0.2764" rpy="-1.5781 -0.91737 1.5766" axis="${wheel_axis_right}" inertial_xyz="-4.8659E-06 -8.069E-06 -0.034709" inertial_rpy="0 0 0"/>
 </robot>

File: AutoNav_Mission_2026/src/maya_description/urdf/sensors_frames.xacro (robot description, xacro)
@@ -25,7 +25,5 @@
         <cylinder radius="0.05" length="0.05"/>
       </geometry>
-      <material name="black">
-        <color rgba="0 0 0 1"/>
-      </material>
+      <material name="sensors"/>
     </visual>
   </link>
@@ -47,6 +45,7 @@
       <origin xyz="0 0 0" rpy="0 0 0"/>
       <geometry>
-        <box size="0.003 0.026 0.0044"/>
+        <box size="0.02 0.14 0.05"/>
       </geometry>
+      <material name="sensors"/>
     </visual>
     <collision>
@@ -65,5 +64,5 @@
     <parent link="base_link"/>
     <child link="camera_link"/>
-    <origin xyz="0 -0.30 0.10" rpy="0 0 ${-half_pi}"/>
+    <origin xyz="0 -0.556 0.03" rpy="0 0 ${-half_pi}"/>
   </joint>
   <link name="camera_depth_frame"/>
