Commit message: Fix: Corrección de rotación del punto de origen del brazo sobre maya a -pi/2 para que se coloque en la posición correspondiente, además de integrar el script para escuchar a los motores del brazo y la simulación funcione correctamente

File: src/maya_description/urdf/maya_arm_mount.xacro (robot description, xacro)
@@ -34,5 +34,5 @@
       <parent link="maya_arm_mount" />
       <child link="arm_base_link" />
-      <origin xyz="${arm_mount_xyz}" rpy="${arm_mount_rpy}"/>
+      <origin xyz="${arm_mount_xyz}" rpy="0 0 -1.57"/>
     </joint>
 </robot>
